Commit message: changed flying_robot_urdf joint names and fixed some urdf problems

File: src/simulation/robots/flying_robot_urdf/flying_robot_urdf.urdf (robot description, URDF)
Before this commit: robot flying_robot_urdf, 13 links, 12 joints
Links:
- link bigleglb: geometry collision mesh filename=package://simulation/robots/flying_robot_urdf/meshes/bigleg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; visual mesh filename=package://simulation/robots/flying_robot_urdf/meshes/bigleg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
- link rightbehind: mass 0 -> 0.798414527576566
Joints:
- removed joint bigleglb
- removed joint bigleglf
- removed joint biglegrb
- removed joint biglegrf
- removed joint leftbehind
- removed joint leftfront
- removed joint rightbehind
- removed joint rightfront
- removed joint smallleglb
- removed joint smallleglf
- removed joint smalllegrb
- removed joint smalllegrf
- added joint jbigleglb: type continuous, parent leftbehind, child bigleglb, origin xyz=-0.095008 0.024981 -0.0421 rpy=1.5708 0.68715 3.1416, axis 0 0 -1, limit lower=0 upper=0 effort=0 velocity=0
- added joint jbigleglf: type continuous, parent leftfront, child bigleglf, origin xyz=0.095008 -0.02502 -0.0421 rpy=1.5708 0.68715 0, axis 0 0 1, limit lower=0 upper=0 effort=0 velocity=0
- added joint jbiglegrb: type continuous, parent rightbehind, child biglegrb, origin xyz=-0.095008 0.024981 -0.0421 rpy=1.5708 0.68715 3.1416, axis 0 0 -1, limit lower=0 upper=0 effort=0 velocity=0
- added joint jbiglegrf: type continuous, parent rightfront, child biglegrf, origin xyz=0.095008 -0.024981 -0.0421 rpy=1.5708 0.68715 0, axis 0 0 1, limit lower=0 upper=0 effort=0 velocity=0
- added joint jleftbehind: type continuous, parent base_link, child leftbehind, origin xyz=-0.20007 0.20003 -0.0004 rpy=0 0 0, axis 0 0 1, limit lower=0 upper=0 effort=0 velocity=0
- added joint jleftfront: type continuous, parent base_link, child leftfront, origin xyz=0.19991 0.20003 -0.0004 rpy=0 0 0, axis 0 0 1, limit lower=0 upper=0 effort=0 velocity=0
- added joint jrightbehind: type continuous, parent base_link, child rightbehind, origin xyz=-0.20007 -0.19997 -0.0004 rpy=0 0 0, axis 0 0 1, limit lower=0 upper=0 effort=0 velocity=0
- added joint jrightfront: type continuous, parent base_link, child rightfront, origin xyz=0.19991 -0.20001 -0.0004 rpy=0 0 0, axis 0 0 1, limit lower=0 upper=0 effort=0 velocity=0
- added joint jsmallleglb: type continuous, parent bigleglb, child smallleglb, origin xyz=0.35 0 -0.025 rpy=0 0 -1.4916, axis 0 0 -1, limit lower=0 upper=0 effort=0 velocity=0
- added joint jsmallleglf: type continuous, parent bigleglf, child smallleglf, origin xyz=0.35 0 -0.025 rpy=0 0 -1.4916, axis 0 0 1, limit lower=0 upper=0 effort=0 velocity=0
- added joint jsmalllegrb: type continuous, parent biglegrb, child smalllegrb, origin xyz=0.35 0 -0.025 rpy=0 0 -1.4916, axis 0 0 -1, limit lower=0 upper=0 effort=0 velocity=0
- added joint jsmalllegrf: type continuous, parent biglegrf, child smalllegrf, origin xyz=0.35 0 -0.025 rpy=0 0 -1.4916, axis 0 0 1, limit lower=0 upper=0 effort=0 velocity=0

File: src/simulation/robots/flying_robot_urdf/urdf/flying_robot_urdf.urdf (robot description, URDF)
Before this commit: robot flying_robot_urdf, 13 links, 12 joints
Links:
- link rightbehind: mass 0 -> 0.798414527576566
Joints:
- removed joint bigleglb
- removed joint bigleglf
- removed joint biglegrb
- removed joint biglegrf
- removed joint leftbehind
- removed joint leftfront
- removed joint rightbehind
- removed joint rightfront
- removed joint smallleglb
- removed joint smallleglf
- removed joint smalllegrb
- removed joint smalllegrf
- added joint jbigleglb: type continuous, parent leftbehind, child bigleglb, origin xyz=-0.095008 0.024981 -0.0421 rpy=1.5708 0.68715 3.1416, axis 0 0 -1, limit lower=0 upper=0 effort=0 velocity=0
- added joint jbigleglf: type continuous, parent leftfront, child bigleglf, origin xyz=0.095008 -0.02502 -0.0421 rpy=1.5708 0.68715 0, axis 0 0 1, limit lower=0 upper=0 effort=0 velocity=0
- added joint jbiglegrb: type continuous, parent rightbehind, child biglegrb, origin xyz=-0.095008 0.024981 -0.0421 rpy=1.5708 0.68715 3.1416, axis 0 0 -1, limit lower=0 upper=0 effort=0 velocity=0
- added joint jbiglegrf: type continuous, parent rightfront, child biglegrf, origin xyz=0.095008 -0.024981 -0.0421 rpy=1.5708 0.68715 0, axis 0 0 1, limit lower=0 upper=0 effort=0 velocity=0
- added joint jleftbehind: type continuous, parent base_link, child leftbehind, origin xyz=-0.20007 0.20003 -0.0004 rpy=0 0 0, axis 0 0 1, limit lower=0 upper=0 effort=0 velocity=0
- added joint jleftfront: type continuous, parent base_link, child leftfront, origin xyz=0.19991 0.20003 -0.0004 rpy=0 0 0, axis 0 0 1, limit lower=0 upper=0 effort=0 velocity=0
- added joint jrightbehind: type continuous, parent base_link, child rightbehind, origin xyz=-0.20007 -0.19997 -0.0004 rpy=0 0 0, axis 0 0 1, limit lower=0 upper=0 effort=0 velocity=0
- added joint jrightfront: type continuous, parent base_link, child rightfront, origin xyz=0.19991 -0.20001 -0.0004 rpy=0 0 0, axis 0 0 1, limit lower=0 upper=0 effort=0 velocity=0
- added joint jsmallleglb: type continuous, parent bigleglb, child smallleglb, origin xyz=0.35 0 -0.025 rpy=0 0 -1.4916, axis 0 0 -1, limit lower=0 upper=0 effort=0 velocity=0
- added joint jsmallleglf: type continuous, parent bigleglf, child smallleglf, origin xyz=0.35 0 -0.025 rpy=0 0 -1.4916, axis 0 0 1, limit lower=0 upper=0 effort=0 velocity=0
- added joint jsmalllegrb: type continuous, parent biglegrb, child smalllegrb, origin xyz=0.35 0 -0.025 rpy=0 0 -1.4916, axis 0 0 -1, limit lower=0 upper=0 effort=0 velocity=0
- added joint jsmalllegrf: type continuous, parent biglegrf, child smalllegrf, origin xyz=0.35 0 -0.025 rpy=0 0 -1.4916, axis 0 0 1, limit lower=0 upper=0 effort=0 velocity=0

File: src/simulation/robots/flying_robot_urdf/urdf/flying_robot_urdf_collision_optim.urdf (robot description, URDF)
Before this commit: robot flying_robot_urdf, 13 links, 12 joints
Links:
- link rightbehind: mass 0 -> 0.798414527576566
Joints:
- removed joint bigleglb
- removed joint bigleglf
- removed joint biglegrb
- removed joint biglegrf
- removed joint leftbehind
- removed joint leftfront
- removed joint rightbehind
- removed joint rightfront
- removed joint smallleglb
- removed joint smallleglf
- removed joint smalllegrb
- removed joint smalllegrf
- added joint jbigleglb: type continuous, parent leftbehind, child bigleglb, origin xyz=-0.095008 0.024981 -0.0421 rpy=1.5708 0.68715 3.1416, axis 0 0 -1, limit lower=0 upper=0 effort=0 velocity=0
- added joint jbigleglf: type continuous, parent leftfront, child bigleglf, origin xyz=0.095008 -0.02502 -0.0421 rpy=1.5708 0.68715 0, axis 0 0 1, limit lower=0 upper=0 effort=0 velocity=0
- added joint jbiglegrb: type continuous, parent rightbehind, child biglegrb, origin xyz=-0.095008 0.024981 -0.0421 rpy=1.5708 0.68715 3.1416, axis 0 0 -1, limit lower=0 upper=0 effort=0 velocity=0
- added joint jbiglegrf: type continuous, parent rightfront, child biglegrf, origin xyz=0.095008 -0.024981 -0.0421 rpy=1.5708 0.68715 0, axis 0 0 1, limit lower=0 upper=0 effort=0 velocity=0
- added joint jleftbehind: type continuous, parent base_link, child leftbehind, origin xyz=-0.20007 0.20003 -0.0004 rpy=0 0 0, axis 0 0 1, limit lower=0 upper=0 effort=0 velocity=0
- added joint jleftfront: type continuous, parent base_link, child leftfront, origin xyz=0.19991 0.20003 -0.0004 rpy=0 0 0, axis 0 0 1, limit lower=0 upper=0 effort=0 velocity=0
- added joint jrightbehind: type continuous, parent base_link, child rightbehind, origin xyz=-0.20007 -0.19997 -0.0004 rpy=0 0 0, axis 0 0 1, limit lower=0 upper=0 effort=0 velocity=0
- added joint jrightfront: type continuous, parent base_link, child rightfront, origin xyz=0.19991 -0.20001 -0.0004 rpy=0 0 0, axis 0 0 1, limit lower=0 upper=0 effort=0 velocity=0
- added joint jsmallleglb: type continuous, parent bigleglb, child smallleglb, origin xyz=0.35 0 -0.025 rpy=0 0 -1.4916, axis 0 0 -1, limit lower=0 upper=0 effort=0 velocity=0
- added joint jsmallleglf: type continuous, parent bigleglf, child smallleglf, origin xyz=0.35 0 -0.025 rpy=0 0 -1.4916, axis 0 0 1, limit lower=0 upper=0 effort=0 velocity=0
- added joint jsmalllegrb: type continuous, parent biglegrb, child smalllegrb, origin xyz=0.35 0 -0.025 rpy=0 0 -1.4916, axis 0 0 -1, limit lower=0 upper=0 effort=0 velocity=0
- added joint jsmalllegrf: type continuous, parent biglegrf, child smalllegrf, origin xyz=0.35 0 -0.025 rpy=0 0 -1.4916, axis 0 0 1, limit lower=0 upper=0 effort=0 velocity=0
