Commit message: feat: using g1_23dof.xacro instead of urdf

File: src/simulation/robots/g1_description/g1_23dof.urdf (robot description, URDF)
Before this commit: robot g1_23dof, 33 links, 32 joints
Links:
- added link dummy_base_link
Joints:
- added joint base_link_joint: type fixed, parent dummy_base_link, child pelvis, origin xyz=0 0 0 rpy=0 0 0
